File: jarpysdr.brd (EAGLE design)
At the start: 90 x 45 mm, 37 parts, among them IC1 74HC74N, IC2 NE5532N, IC3 7805, IC4 TL072P

Commit message: Final physical layout for fab.
Routing:
- net N$16: track 12.1 -> 12.5 mm, vias 1 -> 0

Commit message: Set up silkscreen.
Parts:
- COUNTER: value 74HC74N -> 74HC74
- IC2: value NE5532N -> NE5532
- IC4: value TL072P -> TL072
- JP1: value M10" -> Si570
- SWITCH: value 74HC4052DIP -> 74HC4052
- VEE-IN: value (none) -> -12v
- moved C14 11.3 mm to (70.5, 7.94), turned to 180 degrees
- moved C7 2.48 mm to (51.1, 27.9), turned to 90 degrees
- renumbered IC1 to COUNTER, U$1 to SWITCH
Routing:
- net +12V: track 101.0 -> 101.9 mm
